File: sdcard_switcher.sch (KiCad schematic (older format))
At the start: 12 parts

Commit message: update,
Parts:
- J1, J2: renamed from J?; footprint (none) -> Connector_PinHeader_1.27mm:PinHeader_1x08_P1.27mm_Vertical
- J3: renamed from J?; footprint (none) -> Connector_PinHeader_1.27mm:PinHeader_1x06_P1.27mm_Vertical
- SDC1: renamed from SDC?; footprint (none) -> footprint-lib:SUNTECH_ST-TF-003A
- U1, U2: renamed from U?; footprint (none) -> Package_SO:TSSOP-16_4.4x5mm_P0.65mm
- gave numbers to parts that had none: 6
Changed lines of the file:
@@
 $EndDescr
 $Comp
-L taobao-components:SN74CBT3257D U?
+L taobao-components:SN74CBT3257D U1
 U 1 1 5C14187E
 P 6500 2400
-F 0 "U?" H 6500 3500 50  0000 C CNN
+F 0 "U1" H 6500 3500 50  0000 C CNN
 F 1 "SN74CBT3257D" H 6500 3400 50  0000 C CNN
-F 2 "" H 6550 2400 50  0001 C CNN
+F 2 "Package_SO:TSSOP-16_4.4x5mm_P0.65mm" H 6550 2400 50  0001 C CNN
 F 3 "" H 6550 2400 50  0001 C CNN
 	1    6500 2400
@@
 $EndComp
 $Comp
-L taobao-components:SN74CBT3257D U?
+L taobao-components:SN74CBT3257D U2
 U 1 1 5C144034
 P 6500 4950
-F 0 "U?" H 6500 6050 50  0000 C CNN
+F 0 "U2" H 6500 6050 50  0000 C CNN
 F 1 "SN74CBT3257D" H 6500 5950 50  0000 C CNN
-F 2 "" H 6550 4950 50  0001 C CNN
+F 2 "Package_SO:TSSOP-16_4.4x5mm_P0.65mm" H 6550 4950 50  0001 C CNN
 F 3 "" H 6550 4950 50  0001 C CNN
 	1    6500 4950
@@
 $EndComp
 $Comp
-L Connector_Generic:Conn_01x08 J?
+L Connector_Generic:Conn_01x08 J1
 U 1 1 5C144389
 P 2150 1950
-F 0 "J?" H 2050 2500 50  0000 C CNN
+F 0 "J1" H 2050 2500 50  0000 C CNN
 F 1 "TO_DUT" H 2050 2400 50  0000 C CNN
-F 2 "" H 2150 1950 50  0001 C CNN
+F 2 "Connector_PinHeader_1.27mm:PinHeader_1x08_P1.27mm_Vertical" H 2150 1950 50  0001 C CNN
 F 3 "~" H 2150 1950 50  0001 C CNN
 	1    2150 1950
@@
 	2350 2350 3200 2350
 $Comp
-L Connector_Generic:Conn_01x08 J?
+L Connector_Generic:Conn_01x08 J2
 U 1 1 5C144617
 P 2150 4800
-F 0 "J?" H 2050 5350 50  0000 C CNN
+F 0 "J2" H 2050 5350 50  0000 C CNN
 F 1 "TO_PC" H 2050 5250 50  0000 C CNN
-F 2 "" H 2150 4800 50  0001 C CNN
+F 2 "Connector_PinHeader_1.27mm:PinHeader_1x08_P1.27mm_Vertical" H 2150 4800 50  0001 C CNN
 F 3 "~" H 2150 4800 50  0001 C CNN
 	1    2150 4800
@@
 	2350 5200 3200 5200
 $Comp
-L taobao-components:TF_CARD_SOCKET,SELF_EJECT SDC?
+L taobao-components:TF_CARD_SOCKET,SELF_EJECT SDC1
 U 1 1 5C144E0A
 P 9750 3250
-F 0 "SDC?" H 10250 3250 50  0000 L CNN
+F 0 "SDC1" H 10250 3250 50  0000 L CNN
 F 1 "TF_CARD_SOCKET,SELF_EJECT" H 10250 3150 50  0000 L CNN
-F 2 "" H 9750 3250 50  0001 C CNN
+F 2 "footprint-lib:SUNTECH_ST-TF-003A" H 9750 3250 50  0001 C CNN
 F 3 "" H 9750 3250 50  0001 C CNN
 	1    9750 3250
@@
 DAT1-Y
 $Comp
-L power:GND #PWR?
+L power:GND #PWR0101
 U 1 1 5C1496D3
 P 9950 4150
-F 0 "#PWR?" H 9950 3900 50  0001 C CNN
+F 0 "#PWR0101" H 9950 3900 50  0001 C CNN
 F 1 "GND" H 10000 3950 50  0000 C CNN
 F 2 "" H 9950 4150 50  0001 C CNN
@@
 	8800 3500 9400 3500
 $Comp
-L power:GND #PWR?
+L power:GND #PWR0102
 U 1 1 5C14A9D6
 P 8600 3450
-F 0 "#PWR?" H 8600 3200 50  0001 C CNN
+F 0 "#PWR0102" H 8600 3200 50  0001 C CNN
 F 1 "GND" H 8650 3250 50  0000 C CNN
 F 2 "" H 8600 3450 50  0001 C CNN
@@
 	8600 3300 9400 3300
 $Comp
-L Connector_Generic:Conn_01x06 J?
+L Connector_Generic:Conn_01x06 J3
 U 1 1 5C14BC23
 P 4250 6700
-F 0 "J?" V 4100 7000 50  0000 L CNN
+F 0 "J3" V 4100 7000 50  0000 L CNN
 F 1 "Conn_01x06" V 4200 7000 50  0000 L CNN
-F 2 "" H 4250 6700 50  0001 C CNN
+F 2 "Connector_PinHeader_1.27mm:PinHeader_1x06_P1.27mm_Vertical" H 4250 6700 50  0001 C CNN
 F 3 "~" H 4250 6700 50  0001 C CNN
 	1    4250 6700
@@
 $EndComp
 $Comp
-L power:GND #PWR?
+L power:GND #PWR0103
 U 1 1 5C14CB77
 P 4750 6400
-F 0 "#PWR?" H 4750 6150 50  0001 C CNN
+F 0 "#PWR0103" H 4750 6150 50  0001 C CNN
 F 1 "GND" H 4800 6200 50  0000 C CNN
 F 2 "" H 4750 6400 50  0001 C CNN
@@
 Connection ~ 4350 5250
 $Comp
-L power:GND #PWR?
+L power:GND #PWR0104
 U 1 1 5C150A1A
 P 5000 5850
-F 0 "#PWR?" H 5000 5600 50  0001 C CNN
+F 0 "#PWR0104" H 5000 5600 50  0001 C CNN
 F 1 "GND" H 5050 5650 50  0000 C CNN
 F 2 "" H 5000 5850 50  0001 C CNN
@@
 $EndComp
 $Comp
-L taobao-r:R103,0603 R?
+L taobao-r:R103,0603 R3
 U 1 1 5C150B0B
 P 5350 5550
-F 0 "R?" H 5450 5600 50  0000 L CNN
+F 0 "R3" H 5450 5600 50  0000 L CNN
 F 1 "R103,0603" H 5450 5550 50  0000 L CNN
 F 2 "Resistor_SMD:R_0603_1608Metric_Pad1.05x0.95mm_HandSolder" H 5350 5550 50  0001 C CNN
@@
 $EndComp
 $Comp
-L taobao-r:R103,0603 R?
+L taobao-r:R103,0603 R4
 U 1 1 5C150B45
 P 5350 5900
-F 0 "R?" H 5450 5950 50  0000 L CNN
+F 0 "R4" H 5450 5950 50  0000 L CNN
 F 1 "R103,0603" H 5450 5900 50  0000 L CNN
 F 2 "Resistor_SMD:R_0603_1608Metric_Pad1.05x0.95mm_HandSolder" H 5350 5900 50  0001 C CNN
@@
 	5600 2800 5900 2800
 $Comp
-L power:VCC #PWR?
+L power:VCC #PWR0105
 U 1 1 5C157149
 P 9150 5000
-F 0 "#PWR?" H 9150 4850 50  0001 C CNN
+F 0 "#PWR0105" H 9150 4850 50  0001 C CNN
 F 1 "VCC" H 9200 5200 50  0000 C CNN
 F 2 "" H 9150 5000 50  0001 C CNN
@@
 $EndComp
 $Comp
-L power:VCC #PWR?
+L power:VCC #PWR0106
 U 1 1 5C15716B
 P 4250 6250
-F 0 "#PWR?" H 4250 6100 50  0001 C CNN
+F 0 "#PWR0106" H 4250 6100 50  0001 C CNN
 F 1 "VCC" H 4300 6450 50  0000 C CNN
 F 2 "" H 4250 6250 50  0001 C CNN
@@
 	4250 6250 4250 6500
 $Comp
-L taobao-r:R102,0603 R?
+L taobao-r:R102,0603 R2
 U 1 1 5C158909
 P 9150 5250
-F 0 "R?" H 9250 5300 50  0000 L CNN
+F 0 "R2" H 9250 5300 50  0000 L CNN
 F 1 "R102,0603" H 9250 5250 50  0000 L CNN
 F 2 "Resistor_SMD:R_0603_1608Metric_Pad1.05x0.95mm_HandSolder" H 9150 5250 50  0001 C CNN
@@
 $EndComp
 $Comp
-L taobao-led:LED_GREEN,0603 D?
+L taobao-led:LED_GREEN,0603 D2
 U 1 1 5C158A7C
 P 9150 5650
-F 0 "D?" V 9200 5550 50  0000 R CNN
+F 0 "D2" V 9200 5550 50  0000 R CNN
 F 1 "LED_GREEN,0603" V 9150 5550 50  0000 R CNN
 F 2 "LED_SMD:LED_0603_1608Metric_Pad1.05x0.95mm_HandSolder" V 9150 5650 50  0001 C CNN
@@
 $EndComp
 $Comp
-L power:GND #PWR?
+L power:GND #PWR0107
 U 1 1 5C158B34
 P 9150 5900
-F 0 "#PWR?" H 9150 5650 50  0001 C CNN
+F 0 "#PWR0107" H 9150 5650 50  0001 C CNN
 F 1 "GND" H 9200 5700 50  0000 C CNN
 F 2 "" H 9150 5900 50  0001 C CNN
@@
 HOSTSELECT
 $Comp
-L taobao-r:R102,0603 R?
+L taobao-r:R102,0603 R1
 U 1 1 5C15D494
 P 8300 5250
-F 0 "R?" H 8400 5300 50  0000 L CNN
+F 0 "R1" H 8400 5300 50  0000 L CNN
 F 1 "R102,0603" H 8400 5250 50  0000 L CNN
 F 2 "Resistor_SMD:R_0603_1608Metric_Pad1.05x0.95mm_HandSolder" H 8300 5250 50  0001 C CNN
@@
 $EndComp
 $Comp
-L taobao-led:LED_ORANGE,0603 D?
+L taobao-led:LED_ORANGE,0603 D1
 U 1 1 5C15D69B
 P 8300 5650
-F 0 "D?" V 8350 5550 50  0000 R CNN
+F 0 "D1" V 8350 5550 50  0000 R CNN
 F 1 "LED_ORANGE,0603" V 8300 5550 50  0000 R CNN
 F 2 "LED_SMD:LED_0603_1608Metric_Pad1.05x0.95mm_HandSolder" V 8300 5650 50  0001 C CNN
@@
 $EndComp
 $Comp
-L power:GND #PWR?
+L power:GND #PWR0108
 U 1 1 5C15D770
 P 8300 5900
-F 0 "#PWR?" H 8300 5650 50  0001 C CNN
+F 0 "#PWR0108" H 8300 5650 50  0001 C CNN
 F 1 "GND" H 8350 5700 50  0000 C CNN
 F 2 "" H 8300 5900 50  0001 C CNN
@@
 	8300 5000 8300 5150
 $Comp
-L power:GND #PWR?
+L power:GND #PWR0109
 U 1 1 5C16244F
 P 3450 5000
-F 0 "#PWR?" H 3450 4750 50  0001 C CNN
+F 0 "#PWR0109" H 3450 4750 50  0001 C CNN
 F 1 "GND" H 3500 4800 50  0000 C CNN
 F 2 "" H 3450 5000 50  0001 C CNN
@@
 	2350 4900 3450 4900
 $Comp
-L power:GND #PWR?
+L power:GND #PWR0110
 U 1 1 5C163E78
 P 3450 2200
-F 0 "#PWR?" H 3450 1950 50  0001 C CNN
+F 0 "#PWR0110" H 3450 1950 50  0001 C CNN
 F 1 "GND" H 3500 2000 50  0000 C CNN
 F 2 "" H 3450 2200 50  0001 C CNN
@@
 	2350 2050 3450 2050
 $Comp
-L power:GND #PWR?
+L power:GND #PWR0111
 U 1 1 5C169BC4
 P 7150 5450
-F 0 "#PWR?" H 7150 5200 50  0001 C CNN
+F 0 "#PWR0111" H 7150 5200 50  0001 C CNN
 F 1 "GND" H 7200 5250 50  0000 C CNN
 F 2 "" H 7150 5450 50  0001 C CNN
@@
 	7150 5350 7050 5350
 $Comp
-L power:GND #PWR?
+L power:GND #PWR0112
 U 1 1 5C16B827
 P 7150 2900
-F 0 "#PWR?" H 7150 2650 50  0001 C CNN
+F 0 "#PWR0112" H 7150 2650 50  0001 C CNN
 F 1 "GND" H 7200 2700 50  0000 C CNN
 F 2 "" H 7150 2900 50  0001 C CNN
@@
 	7150 2800 7050 2800
 $Comp
-L power:VCC #PWR?
+L power:VCC #PWR0113
 U 1 1 5C16D507
 P 7150 5150
-F 0 "#PWR?" H 7150 5000 50  0001 C CNN
+F 0 "#PWR0113" H 7150 5000 50  0001 C CNN
 F 1 "VCC" H 7200 5350 50  0000 C CNN
 F 2 "" H 7150 5150 50  0001 C CNN
@@
 	7150 5250 7050 5250
 $Comp
-L power:VCC #PWR?
+L power:VCC #PWR0114
 U 1 1 5C16F30E
 P 7150 2600
-F 0 "#PWR?" H 7150 2450 50  0001 C CNN
+F 0 "#PWR0114" H 7150 2450 50  0001 C CNN
 F 1 "VCC" H 7200 2800 50  0000 C CNN
 F 2 "" H 7150 2600 50  0001 C CNN

Commit message: update,
Other:
- note added: "!! PULL up resistor handling assumed on the DEST side !!"

Commit message: update,
Parts:
- added JP1: Jumper_NO_Small, Jumper:SolderJumper-2_P1.3mm_Open_TrianglePad1.0x1.5mm, symbol Device:Jumper_NO_Small
Connections:
- net VCC: now also JP1.2
- new net +5V: JP1.1
Changed lines of the file:
@@
 	5600 2800 5900 2800
 $Comp
-L power:VCC #PWR0105
-U 1 1 5C157149
-P 9150 5000
-F 0 "#PWR0105" H 9150 4850 50  0001 C CNN
-F 1 "VCC" H 9200 5200 50  0000 C CNN
-F 2 "" H 9150 5000 50  0001 C CNN
-F 3 "" H 9150 5000 50  0001 C CNN
-	1    9150 5000
-	1    0    0    -1
-$EndComp
-$Comp
 L power:VCC #PWR0106
 U 1 1 5C15716B
@@
 Wire Wire Line
 	7150 2800 7050 2800
-$Comp
-L power:VCC #PWR0113
-U 1 1 5C16D507
-P 7150 5150
-F 0 "#PWR0113" H 7150 5000 50  0001 C CNN
-F 1 "VCC" H 7200 5350 50  0000 C CNN
-F 2 "" H 7150 5150 50  0001 C CNN
-F 3 "" H 7150 5150 50  0001 C CNN
-	1    7150 5150
-	1    0    0    -1
-$EndComp
 Wire Wire Line
 	7150 5150 7150 5250
@@
 Text Notes 1900 4150 0    50   ~ 0
 !! PULL up resistor handling assumed on the DEST side !!
+$Comp
+L power:VCC #PWR0105
+U 1 1 5C157149
+P 9150 5000
+F 0 "#PWR0105" H 9150 4850 50  0001 C CNN
+F 1 "VCC" H 9200 5200 50  0000 C CNN
+F 2 "" H 9150 5000 50  0001 C CNN
+F 3 "" H 9150 5000 50  0001 C CNN
+	1    9150 5000
+	1    0    0    -1
+$EndComp
+$Comp
+L power:VCC #PWR0113
+U 1 1 5C16D507
+P 7150 5150
+F 0 "#PWR0113" H 7150 5000 50  0001 C CNN
+F 1 "VCC" H 7200 5350 50  0000 C CNN
+F 2 "" H 7150 5150 50  0001 C CNN
+F 3 "" H 7150 5150 50  0001 C CNN
+	1    7150 5150
+	1    0    0    -1
+$EndComp
+$Comp
+L power:+5V #PWR0115
+U 1 1 5C165BC2
+P 8450 1150
+F 0 "#PWR0115" H 8450 1000 50  0001 C CNN
+F 1 "+5V" H 8500 1350 50  0000 C CNN
+F 2 "" H 8450 1150 50  0001 C CNN
+F 3 "" H 8450 1150 50  0001 C CNN
+	1    8450 1150
+	1    0    0    -1
+$EndComp
+$Comp
+L power:VCC #PWR0116
+U 1 1 5C165C47
+P 9350 1150
+F 0 "#PWR0116" H 9350 1000 50  0001 C CNN
+F 1 "VCC" H 9400 1350 50  0000 C CNN
+F 2 "" H 9350 1150 50  0001 C CNN
+F 3 "" H 9350 1150 50  0001 C CNN
+	1    9350 1150
+	1    0    0    -1
+$EndComp
+$Comp
+L Device:Jumper_NO_Small JP1
+U 1 1 5C165D90
+P 8850 1300
+F 0 "JP1" H 8850 1500 50  0000 C CNN
+F 1 "Jumper_NO_Small" H 8850 1400 50  0000 C CNN
+F 2 "Jumper:SolderJumper-2_P1.3mm_Open_TrianglePad1.0x1.5mm" H 8850 1300 50  0001 C CNN
+F 3 "~" H 8850 1300 50  0001 C CNN
+	1    8850 1300
+	1    0    0    -1
+$EndComp
+Wire Wire Line
+	8450 1150 8450 1300
+Wire Wire Line
+	8450 1300 8750 1300
+Wire Wire Line
+	8950 1300 9350 1300
+Wire Wire Line
+	9350 1300 9350 1150
 $EndSCHEMATC

Commit message: update,
Connections:
- net DAT-A is gone; now on net DAT3-A: J1.7 (Pin_7)
- net DAT-B is gone; now on net DAT3-B: J2.7 (Pin_7)
Changed lines of the file:
@@
 CMD-A
 Text Label 3200 2250 2    50   ~ 0
-DAT-A
+DAT3-A
 Text Label 3200 2350 2    50   ~ 0
 DAT2-A
@@
 CMD-B
 Text Label 3200 5100 2    50   ~ 0
-DAT-B
+DAT3-B
 Text Label 3200 5200 2    50   ~ 0
 DAT2-B
