File: sdcard_switcher.sch (KiCad schematic (older format))
At the start: 13 parts, among them J1 TO_DUT, J2 TO_PC, J3 Conn_01x06, U1 SN74CBT3257D, U2 SN74CBT3257D

Commit message: update,
Parts:
- J1, J2: footprint Connector_PinHeader_1.27mm:PinHeader_1x08_P1.27mm_Vertical -> Connector_FFC-FPC:TE_84952-8_1x08-1MP_P1.0mm_Horizontal
Connections:
- net CLK-A: now also J1.4 (Pin_4); no longer J1.5 (Pin_5)
- net CMD-A: now also J1.6 (Pin_6); no longer J1.3 (Pin_3)
- net DAT0-A: now also J1.2 (Pin_2); no longer J1.7 (Pin_7)
- net DAT1-A: now also J1.1 (Pin_1); no longer J1.8 (Pin_8)
- net DAT2-A: now also J1.8 (Pin_8); no longer J1.1 (Pin_1)
- net DAT3-A: now also J1.7 (Pin_7); no longer J1.2 (Pin_2)
- net GND: now also J1.3 (Pin_3); no longer J1.6 (Pin_6)
- net VDD-A: now also J1.5 (Pin_5); no longer J1.4 (Pin_4)
Other:
- note added: "reverse the order as the component is on the B.Cu"
Changed lines of the file:
@@
 L Connector_Generic:Conn_01x08 J1
 U 1 1 5C144389
-P 3650 2350
-F 0 "J1" H 3550 2900 50  0000 C CNN
-F 1 "TO_DUT" H 3550 2800 50  0000 C CNN
-F 2 "Connector_PinHeader_1.27mm:PinHeader_1x08_P1.27mm_Vertical" H 3650 2350 50  0001 C CNN
-F 3 "~" H 3650 2350 50  0001 C CNN
-	1    3650 2350
-	1    0    0    -1
+P 3650 2450
+F 0 "J1" H 3550 3000 50  0000 C CNN
+F 1 "TO_DUT" H 3550 2900 50  0000 C CNN
+F 2 "Connector_FFC-FPC:TE_84952-8_1x08-1MP_P1.0mm_Horizontal" H 3650 2450 50  0001 C CNN
+F 3 "~" H 3650 2450 50  0001 C CNN
+	1    3650 2450
+	1    0    0    1
 $EndComp
 Text Label 2600 2750 0    50   ~ 0
@@
 F 0 "J2" H 3350 6250 50  0000 C CNN
 F 1 "TO_PC" H 3350 6150 50  0000 C CNN
-F 2 "Connector_PinHeader_1.27mm:PinHeader_1x08_P1.27mm_Vertical" H 3450 5700 50  0001 C CNN
+F 2 "Connector_FFC-FPC:TE_84952-8_1x08-1MP_P1.0mm_Horizontal" H 3450 5700 50  0001 C CNN
 F 3 "~" H 3450 5700 50  0001 C CNN
 	1    3450 5700
@@
 Wire Wire Line
 	9350 1300 9350 1150
+Text Notes 2250 1900 0    50   ~ 0
+reverse the order as the component is on the B.Cu
 $EndSCHEMATC
