File: _saved_sdcard_switcher.sch (KiCad schematic (older format))
At the start: 13 parts, among them J1 TO_DUT, J2 TO_PC, J3 Conn_01x06, U1 SN74CBT3257D, U2 SN74CBT3257D

Commit message: update,
Parts:
- J1: footprint Connector_PinHeader_1.27mm:PinHeader_1x08_P1.27mm_Vertical -> Connector_FFC-FPC:TE_84952-8_1x08-1MP_P1.0mm_Horizontal
Changed lines of the file:
@@
 F 0 "J1" H 3550 2900 50  0000 C CNN
 F 1 "TO_DUT" H 3550 2800 50  0000 C CNN
-F 2 "Connector_PinHeader_1.27mm:PinHeader_1x08_P1.27mm_Vertical" H 3650 2350 50  0001 C CNN
+F 2 "Connector_FFC-FPC:TE_84952-8_1x08-1MP_P1.0mm_Horizontal" H 3650 2350 50  0001 C CNN
 F 3 "~" H 3650 2350 50  0001 C CNN
 	1    3650 2350
