File: sdcard_switcher.kicad_pcb (KiCad board)
At the start: 2 copper layers, 12 parts, among them J1 TO_DUT, J2 TO_PC, J3 Conn_01x06, U1 SN74CBT3257D, U2 SN74CBT3257D

Commit message: update,
Parts:
- added JP1: Jumper_NO_Small, Jumper:SolderJumper-2_P1.3mm_Open_TrianglePad1.0x1.5mm, F.Cu at (66.5, 15.6)
- R2, SDC1: moved to B.Cu
- moved R3 33.3 mm to (77.6, 34.5), turned to 270 degrees
- moved R4 33.0 mm to (79.2, 34.5), turned to 90 degrees
- moved J2 29.3 mm to (59.9, 16.8), turned to 0 degrees
- moved D2 28.6 mm to (77.2, 16.5), turned to 180 degrees
- moved R2 28.6 mm to (77.2, 16.5), turned to 180 degrees
- moved U2 27.1 mm to (72.8, 32.2), turned to 270 degrees
- moved U1 26.7 mm to (72.8, 22.8), turned to 270 degrees
- moved J1 12.2 mm to (59.9, 29.6), turned to 0 degrees
- moved J3 9.00 mm to (75.8, 40.2), turned to 270 degrees
- moved R1 6.09 mm to (65.7, 39.8), turned to 90 degrees
- moved D1 5.44 mm to (67.3, 39.8), turned to 90 degrees
- moved SDC1 4.80 mm to (70.2, 26.5), turned to 270 degrees
Routing:
- net /DAT0-A: track 13.6 -> 31.9 mm, vias 0 -> 1
- net /DAT2-A: track 27.6 -> 14.0 mm, vias 1 -> 0
- net /CLK-A: track 11.4 -> 21.5 mm
- net /HOSTSELECT: track 48.5 -> 39.4 mm, vias 2 -> 4
- net /VDD-A: track 25.6 -> 16.7 mm
- net /CMD-Y: track 16.3 -> 7.69 mm, vias 2 -> 1
- net /DAT1-Y: track 18.1 -> 10.3 mm, vias 0 -> 1
- net /DAT1-B: track 9.98 -> 17.6 mm, vias 0 -> 1
- net /CMD-B: track 11.0 -> 17.7 mm
- net /DAT0-Y: track 17.1 -> 11.2 mm, vias 2 -> 1
- net /CMD-A: track 22.6 -> 17.1 mm, vias 1 -> 2
- net /DAT2-B: track 23.0 -> 19.7 mm, vias 1 -> 0
- net GND: track 146.0 -> 143.0 mm, vias 0 -> 2
- net /VDD-B: track 17.2 -> 20.1 mm
- net VCC: track 49.4 -> 51.3 mm, vias 0 -> 3
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Other:
- board outline added: 30 x 35 mm
- net class .75 added: clearance 0.2, trace_width 0.4, via_dia 0.8, via_drill 0.4
- net class Default: trace_width 0.25 -> 0.4

Commit message: update,
Parts:
- J1: footprint Connector_PinHeader_1.27mm:PinHeader_1x08_P1.27mm_Vertical -> Connector_FFC-FPC:TE_84952-8_1x08-1MP_P1.0mm_Horizontal
- moved D1 8.79 mm to (75.9, 41.6), turned to 270 degrees
- moved R1 8.79 mm to (74.3, 41.6), turned to 270 degrees
- moved R3 8.08 mm to (79.3, 26.6)
- moved R4 8.08 mm to (80.9, 26.6)
- moved J1 7.27 mm to (59.7, 36.9), turned to 270 degrees
- moved U2 2.71 mm to (70.3, 31.1), turned to 180 degrees
- moved U1 2.52 mm to (70.3, 23.1), turned to 180 degrees
- moved SDC1 2.35 mm to (72.5, 26.0)
- moved J3 2.00 mm to (75.9, 38.2)
- moved D2 1.86 mm to (75.7, 15.4)
- moved JP1 1.86 mm to (68.0, 14.5)
- moved R2 1.86 mm to (75.7, 15.4)
Connections:
- J1 pad 1: /DAT1-A -> /DAT2-A
- J1 pad 2: /DAT0-A -> /DAT3-A
- J1 pad 3: /CLK-A -> /CMD-A
- J1 pad 5: GND -> /CLK-A
- J1 pad 6: /CMD-A -> GND
- J1 pad 7: /DAT-A -> /DAT0-A
- J1 pad 8: /DAT2-A -> /DAT1-A
- J2 pad 1: /DAT1-B -> /DAT2-B
- J2 pad 2: /DAT0-B -> /DAT3-B
- J2 pad 3: /CLK-B -> /CMD-B
- J2 pad 5: GND -> /CLK-B
- J2 pad 6: /CMD-B -> GND
- J2 pad 7: /DAT-B -> /DAT0-B
- J2 pad 8: /DAT2-B -> /DAT1-B
- U1 pad 10: GND -> /CMD-B
- U1 pad 11: GND -> /CMD-A
- U1 pad 12: /CLK-Y -> /VDD-Y
- U1 pad 13: /CLK-B -> /VDD-B
- U1 pad 14: /CLK-A -> /VDD-A
- U1 pad 2: /DAT1-A -> /DAT2-A
- U1 pad 3: /DAT1-B -> /DAT2-B
- U1 pad 4: /DAT1-Y -> /DAT2-Y
- U1 pad 5: /DAT0-A -> /DAT3-A
- U1 pad 6: /DAT0-B -> /DAT3-B
- U1 pad 7: /DAT0-Y -> /DAT3-Y
- U1 pad 9: Net-(U1-Pad9) -> /CMD-Y
- U2 pad 10: /DAT2-B -> /DAT0-B
- U2 pad 11: /DAT2-A -> /DAT0-A
- U2 pad 12: /DAT3-Y -> /DAT1-Y
- U2 pad 13: /DAT3-B -> /DAT1-B
- U2 pad 14: /DAT3-A -> /DAT1-A
- U2 pad 2: /VDD-A -> /CLK-A
- U2 pad 3: /VDD-B -> /CLK-B
- U2 pad 4: /VCC-Y -> /CLK-Y
- U2 pad 5: /CMD-A -> GND
- U2 pad 6: /CMD-B -> GND
- U2 pad 7: /CMD-Y -> Net-(U2-Pad7)
- U2 pad 9: /DAT2-Y -> /DAT0-Y
Routing:
- net GND: track 143.0 -> 109.4 mm
- net /DAT3-A: track 0.00 -> 27.4 mm, vias 0 -> 2
- net /VDD-A: track 16.7 -> 42.9 mm, vias 1 -> 0
- net /CMD-A: track 17.1 -> 37.6 mm, vias 2 -> 0
- net /DAT0-A: track 31.9 -> 13.3 mm, vias 1 -> 0
- net /DAT3-B: track 0.00 -> 18.3 mm, vias 0 -> 1
- net /HOSTSELECT: track 39.4 -> 23.0 mm, vias 4 -> 0
- net /OE: track 19.8 -> 33.6 mm
- net VCC: track 51.3 -> 63.1 mm, vias 3 -> 2
- net /VDD-B: track 20.1 -> 8.80 mm
- net /DAT1-A: track 22.6 -> 12.2 mm, vias 1 -> 0
- net /CMD-B: track 17.7 -> 8.41 mm
- net /VDD-Y: track 0.00 -> 7.11 mm, vias 0 -> 1
- net /CLK-B: track 17.4 -> 24.2 mm, vias 0 -> 1
- net /DAT1-Y: track 10.3 -> 16.7 mm
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
Commit message: update,
Parts:
- J1: moved to B.Cu
- J2: footprint Connector_PinHeader_1.27mm:PinHeader_1x08_P1.27mm_Vertical -> Connector_FFC-FPC:TE_84952-8_1x08-1MP_P1.0mm_Horizontal
- R2: moved to F.Cu
- moved JP1 34.2 mm to (84.6, 44.4)
- moved R2 30.5 mm to (81.2, 45.4), turned to 0 degrees
- moved D2 29.0 mm to (81.3, 43.9), turned to 0 degrees
- moved R4 22.1 mm to (77.8, 48.5), turned to 0 degrees
- moved R3 20.4 mm to (77.8, 47.0), turned to 0 degrees
- moved J2 15.4 mm to (57.6, 32.0), turned to 270 degrees
- moved J1 7.79 mm to (57.6, 29.4), turned to 90 degrees
- moved J3 6.22 mm to (74.6, 44.3), turned to 0 degrees
- moved U2 5.94 mm to (71.0, 37.0)
- moved R1 5.22 mm to (77.8, 45.4), turned to 0 degrees
- moved SDC1 4.12 mm to (73.5, 30.0)
- moved D1 3.02 mm to (77.9, 43.9), turned to 0 degrees
- moved U1 2.79 mm to (71.0, 25.8), turned to 0 degrees
Connections:
- J1 pad 1: /DAT2-A -> /DAT1-A
- J1 pad 2: /DAT3-A -> /DAT0-A
- J1 pad 3: /CMD-A -> GND
- J1 pad 4: /VDD-A -> /CLK-A
- J1 pad 5: /CLK-A -> /VDD-A
- J1 pad 6: GND -> /CMD-A
- J1 pad 7: /DAT0-A -> /DAT3-A
- J1 pad 8: /DAT1-A -> /DAT2-A
Routing:
- net GND: track 109.4 -> 63.6 mm, vias 2 -> 3
- net VCC: track 63.1 -> 22.0 mm, vias 2 -> 0
- net /VDD-A: track 42.9 -> 17.2 mm, vias 0 -> 1
- net /CMD-A: track 37.6 -> 17.9 mm, vias 0 -> 1
- net /DAT3-A: track 27.4 -> 9.17 mm, vias 2 -> 1
- net /OE: track 33.6 -> 20.0 mm
- net /VDD-B: track 8.80 -> 22.2 mm
- net /CLK-Y: track 10.2 -> 22.2 mm
- net /DAT2-B: track 22.0 -> 10.2 mm, vias 1 -> 0
- net /CMD-B: track 8.41 -> 19.2 mm
- net /DAT2-A: track 18.9 -> 9.36 mm, vias 2 -> 1
- net /DAT3-B: track 18.3 -> 9.83 mm, vias 1 -> 0
- net /HOSTSELECT: track 23.0 -> 27.0 mm
- net /CMD-Y: track 10.9 -> 7.53 mm
- net /DAT3-Y: track 10.8 -> 7.51 mm
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Other:
- board outline removed
